File: dock/ZSWatch-Dock.kicad_pcb (KiCad board)
At the start: 4 copper layers, 80 x 48 mm, 73 parts, among them IC401 TLV70218_SOT23-5, IC402 USBLC6-2P6, IC403 FT230XQ, IC404 MIC5219-3.3YM5, IC405 TXB0304RUT, IC406 USBLC6-2P6, IC407 USB2512BT, IC408 USBLC6-2P6, IC409 MIC2026-1xM, J402 Voltage, Q401 BSH205G2AR, SW401 Charge, X401 Debug, X402 UART, X403 Host, X404 Device, X405 Current, Y401 24 MHz

Commit message: Update outputs (release)
Other:
- board text added: "0.035mm (1.00oz)"
- board text added: "0.1855mm"
- board text added: "0.23mm"
- board text added: "Inner1"
- board text added: "Inner2"
- board text added: "Plane"
- board text added: "Prepreg"
- board text added: "Total thickness: 0.761mm"
- board text removed: "0.035mm (1oz)"
- board text removed: "1.51mm"
- board text removed: "Total thickness: 1.6mm"
